Commit message: 修改了重量

File: urdf/mid360.xacro (robot description, xacro)
@@ -8,5 +8,5 @@
   <xacro:property name="noise_mean" value="0.0"/>
   <xacro:property name="noise_stddev" value="0.01"/>
-  <xacro:property name="mass" value="0.4" />
+  <xacro:property name="mass" value="0.004" />
   <xacro:property name="length" value="0.1" />
   <xacro:property name="width" value="0.06" />
